File: LCD-encoder for prototyping/LCD-encoder for prototyping.kicad_pcb (KiCad board)
At the start: 2 copper layers, 40 parts, among them J1 3v3 select, J2 CONN_01X10, J3 CONN_01X04, J4 CONN_01X02, J5 SDA_jumper, J6 SCL_jumper, Q1 2N7002, Q2 2N7002, SW1 Rotary_Encoder_Switch, SW2 Rotary_Encoder_Switch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

Commit message: Add files via upload
Parts:
- added C7: 1u, Capacitors_SMD:C_0805_HandSoldering, F.Cu at (123.2, 69.8)
- added C8: 1u, Capacitors_SMD:C_0805_HandSoldering, F.Cu at (128.3, 88.9)
- SW1, SW2: moved to B.Cu
- moved J3 91.6 mm to (163.8, 78.5)
- moved R8 79.2 mm to (149.9, 47.0), turned to 90 degrees
- moved R10 78.7 mm to (141.0, 50.8)
- moved SW2 68.1 mm to (160.0, 50.0)
- moved R9 67.8 mm to (141.0, 41.9), turned to 180 degrees
- moved J4 65.0 mm to (163.8, 69.8)
- moved R6 56.7 mm to (121.9, 41.9)
- moved SW1 55.9 mm to (100.0, 50.0)
- moved R3 54.9 mm to (121.9, 57.1)
- moved Q2 54.2 mm to (154.7, 88.0)
- moved R4 53.3 mm to (121.9, 49.5), turned to 180 degrees
- moved R5 52.9 mm to (111.8, 47.0), turned to 90 degrees
- moved R1 51.5 mm to (111.8, 54.6), turned to 270 degrees
- moved R16 49.5 mm to (154.9, 83.8)
- moved D2 49.3 mm to (121.9, 53.3), turned to 180 degrees
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Routing:
- net VCC: track 0.00 -> 150.6 mm, vias 0 -> 4
- net VDD: track 0.00 -> 102.7 mm
- net Net-(J2-Pad1): track 0.00 -> 85.5 mm
- net Net-(C8-Pad2): track 0.00 -> 49.6 mm
- net Net-(C2-Pad2): track 0.00 -> 49.2 mm
- net Net-(D4-Pad2): track 0.00 -> 46.5 mm
- net Net-(C3-Pad2): track 0.00 -> 37.9 mm
- net Net-(C1-Pad2): track 0.00 -> 35.6 mm
- net Net-(D6-Pad2): track 0.00 -> 34.7 mm
- net Net-(D5-Pad2): track 0.00 -> 34.4 mm
- net enc1BTN: track 0.00 -> 32.3 mm
- net Net-(D2-Pad2): track 0.00 -> 31.7 mm
- net enc1B: track 0.00 -> 31.3 mm
- net Net-(D3-Pad2): track 0.00 -> 28.3 mm
- net Net-(D1-Pad2): track 0.00 -> 27.2 mm
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- added copper zone on F.Cu, net GND
Other:
- net class Default: clearance 0.2 -> 0.3; trace_width 0.25 -> 0.5; via_dia 0.6 -> 1.2; via_drill 0.4 -> 0.8
- rule trace_clearance: 0.2 -> 0.3

Commit message: Add files via upload
Parts:
- added REF**: C_0805_HandSoldering, Capacitors_SMD:C_0805_HandSoldering, F.Cu at (142.2, 71.8)
- J3: value CONN_01X04 -> LCD_i2c
- moved C8 41.4 mm to (141.0, 49.5), turned to 180 degrees
- moved C2 31.9 mm to (120.7, 49.5), turned to 0 degrees
- moved C3 19.1 mm to (141.0, 59.7), turned to 180 degrees
- moved C1 14.2 mm to (120.7, 59.7), turned to 0 degrees
- moved R3 5.24 mm to (120.7, 62.2)
- moved D1 5.16 mm to (121.0, 66.0)
- moved U1 4.02 mm to (127.0, 73.7)
- moved D6 3.81 mm to (141.0, 66.0)
- moved R12 3.81 mm to (141.0, 62.2)
- moved D2 2.84 mm to (120.7, 55.9)
- moved R4 2.84 mm to (120.7, 52.1)
- moved C4 2.82 mm to (142.2, 69.8), turned to 180 degrees
- moved R11 2.54 mm to (149.9, 61.0), turned to 270 degrees
- moved R5 2.54 mm to (111.8, 44.5), turned to 270 degrees
- moved R8 2.54 mm to (149.9, 44.5), turned to 270 degrees
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Routing:
- net VCC: track 150.6 -> 258.2 mm
- net Net-(J2-Pad2): track 0.00 -> 89.6 mm, vias 0 -> 2
- net enc2B: track 0.00 -> 76.8 mm, vias 0 -> 2
- net enc2BTN: track 0.00 -> 76.5 mm, vias 0 -> 2
- net enc2A: track 0.00 -> 64.6 mm, vias 0 -> 2
- net enc1A: track 0.00 -> 34.5 mm
- net Net-(D4-Pad2): track 46.5 -> 23.9 mm
- net Net-(D5-Pad2): track 34.4 -> 20.1 mm
- net enc1B: track 31.3 -> 45.6 mm, vias 0 -> 2
- net GND: track 0.00 -> 10.1 mm, vias 0 -> 2
- net Net-(C2-Pad2): track 49.2 -> 58.8 mm
- net VDD: track 102.7 -> 112.0 mm, vias 0 -> 3
- net Net-(D6-Pad2): track 34.7 -> 27.2 mm
- net Net-(C8-Pad2): track 49.6 -> 56.7 mm
- net Net-(C1-Pad2): track 35.6 -> 42.2 mm
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- added copper zone on B.Cu, net GND
Other:
- board outline added: 79.4 x 59.1 mm
- board text added: "SCL"
- board text added: "SDA"
- board text added: "Vsel"

Commit message: V2
Parts:
- removed J4: CONN_01X02, Pin_Headers:Pin_Header_Straight_1x02_Pitch2.54mm
- removed J5: SDA_jumper, Pin_Headers:Pin_Header_Straight_1x02_Pitch2.54mm
- removed J6: SCL_jumper, Pin_Headers:Pin_Header_Straight_1x02_Pitch2.54mm
- removed the REF** at (142.2, 71.8)
- removed SW1, SW2: Rotary_Encoder_Switch, sparkfun:SF-ROTARY-ENCODER
- added C11: 0,1u, Capacitors_SMD:C_0805_HandSoldering, F.Cu at (115.5, 77.5)
- added REF**: 1U, Capacitors_SMD:C_0805_HandSoldering, F.Cu at (128.9, 92.1)
- added REF**: 0,1U, Capacitors_SMD:C_0805_HandSoldering, F.Cu at (131.4, 92.1)
- added REF**: 0,1U, Capacitors_SMD:C_0805_HandSoldering, F.Cu at (148.0, 94.0)
- added REF**: 1U, Capacitors_SMD:C_0805_HandSoldering, F.Cu at (151.1, 94.0)
- added ROT1: ROTARY-ENCODER-Ebay, Libs:ROTARY-ENCODER-Ebay, F.Cu at (100.0, 50.0)
- added ROT2: ROTARY-ENCODER-Ebay, Libs:ROTARY-ENCODER-Ebay, F.Cu at (160.0, 50.0)
- D1, D2, D3, D4, D5, D6: footprint Diodes_SMD:D_MELF-RM10_Universal_Handsoldering -> Diodes_SMD:D_MiniMELF_Handsoldering
- Q1, Q2: footprint TO_SOT_Packages_SMD:SOT-23 -> TO_SOT_Packages_SMD:SOT-23_Handsoldering
- moved C4 16.1 mm to (137.2, 54.6), turned to 0 degrees
- moved C7 15.3 mm to (121.9, 54.6), turned to 180 degrees
- moved R14 15.3 mm to (153.7, 88.9)
- moved D1 14.6 mm to (116.8, 52.1)
- moved D6 14.0 mm to (142.2, 52.1)
- moved U1 13.4 mm to (120.3, 85.2), turned to 90 degrees
- moved R4 13.3 mm to (116.8, 64.8)
- moved R10 12.8 mm to (142.2, 64.8)
- moved R16 12.2 mm to (167.0, 81.9), turned to 90 degrees
- moved C5 11.4 mm to (102.9, 92.1)
- moved U2 11.4 mm to (110.5, 89.5)
- moved C6 11.2 mm to (102.9, 89.5)
- moved R15 10.2 mm to (148.6, 78.7)
- moved R1 10.2 mm to (102.9, 49.5), turned to 90 degrees
- moved Q2 10.2 mm to (153.4, 79.1)
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Connections:
- net /SCL renamed /SCLlvl
- net /SDA renamed /SDAlvl
- J2 pad 1: Net-(J2-Pad1) -> SCL
- J2 pad 2: Net-(J2-Pad2) -> SDA
- J3 pad 2: Net-(J3-Pad2) -> VDD
- Q1 pad 2: Net-(J5-Pad1) -> SDA
- Q2 pad 2: Net-(J6-Pad1) -> SCL
- R13 pad 2: Net-(J5-Pad1) -> SDA
- R15 pad 2: Net-(J6-Pad1) -> SCL
- U1 pad 10: enc2BTN -> enc2B
- U1 pad 11: Net-(C3-Pad2) -> Net-(C4-Pad2)
- U1 pad 12: enc2B -> enc2BTN
- U1 pad 13: Net-(C4-Pad2) -> Net-(C3-Pad2)
- U1 pad 3: Net-(C1-Pad2) -> Net-(C2-Pad2)
- U1 pad 4: enc1BTN -> enc1B
- U1 pad 5: Net-(C2-Pad2) -> Net-(C1-Pad2)
- U1 pad 6: enc1B -> enc1BTN
Routing:
- net SCL: track 0.00 -> 90.4 mm, vias 0 -> 2
- net Net-(J2-Pad2): track 89.6 -> 0.00 mm, vias 2 -> 0
- net Net-(J2-Pad1): track 86.0 -> 0.00 mm, vias 2 -> 0
- net SDA: track 0.00 -> 82.9 mm, vias 0 -> 2
- net enc2BTN: track 76.5 -> 35.4 mm, vias 2 -> 0
- net enc2B: track 76.8 -> 39.6 mm, vias 2 -> 0
- net VCC: track 258.2 -> 233.9 mm, vias 4 -> 0
- net enc2A: track 64.6 -> 44.3 mm, vias 2 -> 0
- net Net-(C7-Pad2): track 22.1 -> 40.7 mm, vias 0 -> 1
- net Net-(D5-Pad2): track 20.1 -> 36.0 mm
- net Net-(D1-Pad2): track 29.0 -> 14.2 mm
- net Net-(D3-Pad2): track 26.8 -> 13.2 mm
- net Net-(C8-Pad2): track 56.7 -> 44.5 mm
- net Net-(D6-Pad2): track 27.2 -> 15.1 mm
- net Net-(J3-Pad2): track 11.4 -> 0.00 mm
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Other:
- board size 79.4 x 59.1 mm -> 78.7 x 59.1 mm
- net class Default: via_dia 1.2 -> 1.5
- board text removed: "SCL"
- board text removed: "SDA"
- board text removed: "Vsel"
