File: LCD-encoder for prototyping/LCD-encoder for prototyping.sch (KiCad schematic (older format))
At the start: 40 parts, among them J1 3v3 select, J2 CONN_01X10, J3 CONN_01X04, J4 CONN_01X02, J5 SDA_jumper, J6 SCL_jumper, Q1 2N7002, Q2 2N7002, SW1 Rotary_Encoder_Switch, SW2 Rotary_Encoder_Switch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

Commit message: Add files via upload
Parts:
- added C7, C8: 1u, Capacitors_SMD:C_0805_HandSoldering, symbol C
- Q1, Q2: symbol 2N7002 -> 2N7002-RESCUE-LCD-encoder_for_prototyping
- U2: symbol LM1117-3.3 -> LM1117-3.3-RESCUE-LCD-encoder_for_prototyping
Connections:
- net GND: now also C7.1, C8.1
- net at D4.1 (K), R9.2, U1.9: now also C8.2
- net at D1.1 (K), R3.2, U1.1: now also C7.2
Changed lines of the file:
@@
 EESchema Schematic File Version 2
+LIBS:LCD-encoder for prototyping-rescue
 LIBS:power
 LIBS:device
@@
 LIBS:contrib
 LIBS:valves
-LIBS:4000-ic
-LIBS:7400-ic
-LIBS:analog-ic
-LIBS:avr-mcu
-LIBS:bluegiga
-LIBS:connector
-LIBS:diode-inc-ic
-LIBS:freescale-ic
-LIBS:ftdi-ic
-LIBS:led
-LIBS:maxim-ic
-LIBS:micrel-ic
-LIBS:microchip-ic
-LIBS:nxp-ic
-LIBS:on-semi-ic
-LIBS:regulator
-LIBS:rohm
-LIBS:sharp-relay
-LIBS:sparkfun
-LIBS:standard
-LIBS:stmicro-mcu
-LIBS:ti-ic
-LIBS:transistor
-LIBS:uln-ic
 LIBS:LCD-encoder for prototyping-cache
 EELAYER 25 0
@@
 $EndComp
 $Comp
-L GND #PWR25
+L GND #PWR20
 U 1 1 59AD8FF2
 P 4350 6000
-F 0 "#PWR25" H 4350 5750 50  0001 C CNN
+F 0 "#PWR20" H 4350 5750 50  0001 C CNN
 F 1 "GND" H 4350 5850 50  0000 C CNN
 F 2 "" H 4350 6000 50  0001 C CNN
@@
 $EndComp
 $Comp
-L GND #PWR23
+L GND #PWR15
 U 1 1 59ADA6B8
 P 3450 5350
-F 0 "#PWR23" H 3450 5100 50  0001 C CNN
+F 0 "#PWR15" H 3450 5100 50  0001 C CNN
 F 1 "GND" H 3450 5200 50  0000 C CNN
 F 2 "" H 3450 5350 50  0001 C CNN
@@
 $EndComp
 $Comp
-L VCC #PWR20
+L VCC #PWR16
 U 1 1 59ADB86E
 P 3500 4850
-F 0 "#PWR20" H 3500 4700 50  0001 C CNN
+F 0 "#PWR16" H 3500 4700 50  0001 C CNN
 F 1 "VCC" H 3500 5000 50  0000 C CNN
 F 2 "" H 3500 4850 50  0001 C CNN
@@
 $EndComp
 $Comp
-L GND #PWR26
+L GND #PWR7
 U 1 1 59ADBA94
 P 2650 6900
-F 0 "#PWR26" H 2650 6650 50  0001 C CNN
+F 0 "#PWR7" H 2650 6650 50  0001 C CNN
 F 1 "GND" H 2650 6750 50  0000 C CNN
 F 2 "" H 2650 6900 50  0001 C CNN
@@
 	3600 6000 3200 6000
 $Comp
-L VCC #PWR24
+L VCC #PWR12
 U 1 1 59ADC41B
 P 3200 5650
-F 0 "#PWR24" H 3200 5500 50  0001 C CNN
+F 0 "#PWR12" H 3200 5500 50  0001 C CNN
 F 1 "VCC" H 3200 5800 50  0000 C CNN
 F 2 "" H 3200 5650 50  0001 C CNN
@@
 $EndComp
 $Comp
-L VCC #PWR7
+L VCC #PWR17
 U 1 1 59ADD977
 P 4200 1650
-F 0 "#PWR7" H 4200 1500 50  0001 C CNN
+F 0 "#PWR17" H 4200 1500 50  0001 C CNN
 F 1 "VCC" H 4200 1800 50  0000 C CNN
 F 2 "" H 4200 1650 50  0001 C CNN
@@
 $EndComp
 $Comp
-L GND #PWR12
+L GND #PWR18
 U 1 1 59ADD97D
 P 4250 3050
-F 0 "#PWR12" H 4250 2800 50  0001 C CNN
+F 0 "#PWR18" H 4250 2800 50  0001 C CNN
 F 1 "GND" H 4250 2900 50  0000 C CNN
 F 2 "" H 4250 3050 50  0001 C CNN
@@
 $EndComp
 $Comp
-L GND #PWR9
+L GND #PWR13
 U 1 1 59ADD989
 P 3350 2400
-F 0 "#PWR9" H 3350 2150 50  0001 C CNN
+F 0 "#PWR13" H 3350 2150 50  0001 C CNN
 F 1 "GND" H 3350 2250 50  0000 C CNN
 F 2 "" H 3350 2400 50  0001 C CNN
@@
 $EndComp
 $Comp
-L VCC #PWR8
+L VCC #PWR14
 U 1 1 59ADD9A2
 P 3400 1900
-F 0 "#PWR8" H 3400 1750 50  0001 C CNN
+F 0 "#PWR14" H 3400 1750 50  0001 C CNN
 F 1 "VCC" H 3400 2050 50  0000 C CNN
 F 2 "" H 3400 1900 50  0001 C CNN
@@
 $EndComp
 $Comp
-L GND #PWR16
+L GND #PWR6
 U 1 1 59ADD9B4
 P 2550 3950
-F 0 "#PWR16" H 2550 3700 50  0001 C CNN
+F 0 "#PWR6" H 2550 3700 50  0001 C CNN
 F 1 "GND" H 2550 3800 50  0000 C CNN
 F 2 "" H 2550 3950 50  0001 C CNN
@@
 	3500 3050 3100 3050
 $Comp
-L VCC #PWR10
+L VCC #PWR11
 U 1 1 59ADD9E1
 P 3100 2700
-F 0 "#PWR10" H 3100 2550 50  0001 C CNN
+F 0 "#PWR11" H 3100 2550 50  0001 C CNN
 F 1 "VCC" H 3100 2850 50  0000 C CNN
 F 2 "" H 3100 2700 50  0001 C CNN
@@
 	2500 3100 2500 3350
 $Comp
-L GND #PWR15
+L GND #PWR22
 U 1 1 59ADE53B
 P 7650 3100
-F 0 "#PWR15" H 7650 2850 50  0001 C CNN
+F 0 "#PWR22" H 7650 2850 50  0001 C CNN
 F 1 "GND" H 7650 2950 50  0000 C CNN
 F 2 "" H 7650 3100 50  0001 C CNN
@@
 enc2B
 $Comp
-L LM1117-3.3 U2
+L LM1117-3.3-RESCUE-LCD-encoder_for_prototyping U2
 U 1 1 59AD887C
 P 1650 1100
@@
 $EndComp
 $Comp
-L VDD #PWR11
+L VDD #PWR21
 U 1 1 59AD924F
 P 7100 2900
-F 0 "#PWR11" H 7100 2750 50  0001 C CNN
+F 0 "#PWR21" H 7100 2750 50  0001 C CNN
 F 1 "VDD" H 7100 3050 50  0000 C CNN
 F 2 "" H 7100 2900 50  0001 C CNN
@@
 Connection ~ 2100 1100
 $Comp
-L GND #PWR4
+L GND #PWR3
 U 1 1 59ADA7A1
 P 1650 1450
-F 0 "#PWR4" H 1650 1200 50  0001 C CNN
+F 0 "#PWR3" H 1650 1200 50  0001 C CNN
 F 1 "GND" H 1650 1300 50  0000 C CNN
 F 2 "" H 1650 1450 50  0001 C CNN
@@
 	1650 1450 1650 1400
 $Comp
-L GND #PWR5
+L GND #PWR2
 U 1 1 59ADA88F
 P 1200 1500
-F 0 "#PWR5" H 1200 1250 50  0001 C CNN
+F 0 "#PWR2" H 1200 1250 50  0001 C CNN
 F 1 "GND" H 1200 1350 50  0000 C CNN
 F 2 "" H 1200 1500 50  0001 C CNN
@@
 $EndComp
 $Comp
-L GND #PWR6
+L GND #PWR4
 U 1 1 59ADA900
 P 2100 1550
-F 0 "#PWR6" H 2100 1300 50  0001 C CNN
+F 0 "#PWR4" H 2100 1300 50  0001 C CNN
 F 1 "GND" H 2100 1400 50  0000 C CNN
 F 2 "" H 2100 1550 50  0001 C CNN
@@
 $EndComp
 $Comp
-L VCC #PWR2
+L VCC #PWR9
 U 1 1 59ADAB9E
 P 2900 1200
-F 0 "#PWR2" H 2900 1050 50  0001 C CNN
+F 0 "#PWR9" H 2900 1050 50  0001 C CNN
 F 1 "VCC" H 2900 1350 50  0000 C CNN
 F 2 "" H 2900 1200 50  0001 C CNN
@@
 	2800 1100 2800 1200
 $Comp
-L VDD #PWR3
+L VDD #PWR10
 U 1 1 59ADAC93
 P 3000 1200
-F 0 "#PWR3" H 3000 1050 50  0001 C CNN
+F 0 "#PWR10" H 3000 1050 50  0001 C CNN
 F 1 "VDD" H 3000 1350 50  0000 C CNN
 F 2 "" H 3000 1200 50  0001 C CNN
@@
 SCL
 $Comp
-L GND #PWR22
+L GND #PWR27
 U 1 1 59ADBA81
 P 9900 5300
-F 0 "#PWR22" H 9900 5050 50  0001 C CNN
+F 0 "#PWR27" H 9900 5050 50  0001 C CNN
 F 1 "GND" H 9900 5150 50  0000 C CNN
 F 2 "" H 9900 5300 50  0001 C CNN
@@
 $EndComp
 $Comp
-L VDD #PWR21
+L VDD #PWR28
 U 1 1 59ADBB88
 P 10650 5200
-F 0 "#PWR21" H 10650 5050 50  0001 C CNN
+F 0 "#PWR28" H 10650 5050 50  0001 C CNN
 F 1 "VDD" H 10650 5350 50  0000 C CNN
 F 2 "" H 10650 5200 50  0001 C CNN
@@
 	10400 5200 10650 5200
 $Comp
-L 2N7002 Q1
+L 2N7002-RESCUE-LCD-encoder_for_prototyping Q1
 U 1 1 59ADD065
 P 9400 3500
@@
 	9050 3450 9050 3800
 $Comp
-L VDD #PWR14
+L VDD #PWR26
 U 1 1 59AE518F
 P 9800 3050
-F 0 "#PWR14" H 9800 2900 50  0001 C CNN
+F 0 "#PWR26" H 9800 2900 50  0001 C CNN
 F 1 "VDD" H 9800 3200 50  0000 C CNN
 F 2 "" H 9800 3050 50  0001 C CNN
@@
 	9800 3050 9800 3150
 $Comp
-L VCC #PWR13
+L VCC #PWR24
 U 1 1 59AE585A
 P 9050 3050
-F 0 "#PWR13" H 9050 2900 50  0001 C CNN
+F 0 "#PWR24" H 9050 2900 50  0001 C CNN
 F 1 "VCC" H 9050 3200 50  0000 C CNN
 F 2 "" H 9050 3050 50  0001 C CNN
@@
 	10200 3600 10200 5100
 $Comp
-L 2N7002 Q2
+L 2N7002-RESCUE-LCD-encoder_for_prototyping Q2
 U 1 1 59AE898D
 P 8750 4600
@@
 	8400 4550 8400 4700
 $Comp
-L VDD #PWR18
+L VDD #PWR25
 U 1 1 59AE89A3
 P 9150 4150
-F 0 "#PWR18" H 9150 4000 50  0001 C CNN
+F 0 "#PWR25" H 9150 4000 50  0001 C CNN
 F 1 "VDD" H 9150 4300 50  0000 C CNN
 F 2 "" H 9150 4150 50  0001 C CNN
@@
 	9150 4150 9150 4250
 $Comp
-L VCC #PWR17
+L VCC #PWR23
 U 1 1 59AE89AB
 P 8400 4150
-F 0 "#PWR17" H 8400 4000 50  0001 C CNN
+F 0 "#PWR23" H 8400 4000 50  0001 C CNN
 F 1 "VCC" H 8400 4300 50  0000 C CNN
 F 2 "" H 8400 4150 50  0001 C CNN
@@
 Wire Wire Line
 	9050 3800 8000 3800
+$Comp
+L C C7
+U 1 1 59B1639E
+P 2450 2550
+F 0 "C7" H 2475 2650 50  0000 L CNN
+F 1 "1u" H 2475 2450 50  0000 L CNN
+F 2 "Capacitors_SMD:C_0805_HandSoldering" H 2488 2400 50  0001 C CNN
+F 3 "" H 2450 2550 50  0001 C CNN
+	1    2450 2550
+	-1   0    0    1
+$EndComp
+$Comp
+L GND #PWR5
+U 1 1 59B16466
+P 2450 2800
+F 0 "#PWR5" H 2450 2550 50  0001 C CNN
+F 1 "GND" H 2450 2650 50  0000 C CNN
+F 2 "" H 2450 2800 50  0001 C CNN
+F 3 "" H 2450 2800 50  0001 C CNN
+	1    2450 2800
+	1    0    0    -1
+$EndComp
+$Comp
+L C C8
+U 1 1 59B164FB
+P 2800 5500
+F 0 "C8" H 2825 5600 50  0000 L CNN
+F 1 "1u" H 2825 5400 50  0000 L CNN
+F 2 "Capacitors_SMD:C_0805_HandSoldering" H 2838 5350 50  0001 C CNN
+F 3 "" H 2800 5500 50  0001 C CNN
+	1    2800 5500
+	-1   0    0    1
+$EndComp
+$Comp
+L GND #PWR8
+U 1 1 59B165E2
+P 2800 5700
+F 0 "#PWR8" H 2800 5450 50  0001 C CNN
+F 1 "GND" H 2800 5550 50  0000 C CNN
+F 2 "" H 2800 5700 50  0001 C CNN
+F 3 "" H 2800 5700 50  0001 C CNN
+	1    2800 5700
+	1    0    0    -1
+$EndComp
+Wire Wire Line
+	2800 5350 2800 5250
+Connection ~ 2800 5250
+Wire Wire Line
+	2800 5700 2800 5650
+Wire Wire Line
+	2450 2800 2450 2700
+Wire Wire Line
+	2450 2400 2450 2250
+Connection ~ 2450 2250
 $EndSCHEMATC

Commit message: Add files via upload
Parts:
- J3: value CONN_01X04 -> LCD_i2c
Changed lines of the file:
@@
 LIBS:contrib
 LIBS:valves
+LIBS:4000-ic
+LIBS:7400-ic
+LIBS:analog-ic
+LIBS:avr-mcu
+LIBS:bluegiga
+LIBS:connector
+LIBS:diode-inc-ic
+LIBS:freescale-ic
+LIBS:ftdi-ic
+LIBS:led
+LIBS:maxim-ic
+LIBS:micrel-ic
+LIBS:microchip-ic
+LIBS:nxp-ic
+LIBS:on-semi-ic
+LIBS:regulator
+LIBS:rohm
+LIBS:sharp-relay
+LIBS:sparkfun
+LIBS:standard
+LIBS:stmicro-mcu
+LIBS:ti-ic
+LIBS:transistor
+LIBS:uln-ic
 LIBS:LCD-encoder for prototyping-cache
 EELAYER 25 0
@@
 P 9700 5150
 F 0 "J3" H 9700 5400 50  0000 C CNN
-F 1 "CONN_01X04" V 9800 5150 50  0000 C CNN
+F 1 "LCD_i2c" V 9800 5150 50  0000 C CNN
 F 2 "Pin_Headers:Pin_Header_Straight_1x04_Pitch2.54mm" H 9700 5150 50  0001 C CNN
 F 3 "" H 9700 5150 50  0001 C CNN

Commit message: V2
Parts:
- removed J4: CONN_01X02, Pin_Headers:Pin_Header_Straight_1x02_Pitch2.54mm, symbol CONN_01X02
- removed J5: SDA_jumper, Pin_Headers:Pin_Header_Straight_1x02_Pitch2.54mm, symbol CONN_01X02
- removed J6: SCL_jumper, Pin_Headers:Pin_Header_Straight_1x02_Pitch2.54mm, symbol CONN_01X02
- removed SW1, SW2: Rotary_Encoder_Switch, sparkfun:SF-ROTARY-ENCODER, symbol Rotary_Encoder_Switch
- added C11: 0,1u, Capacitors_SMD:C_0805_HandSoldering, symbol C
- added ROT1, ROT2: ROTARY-ENCODER-Ebay, Libs:ROTARY-ENCODER-Ebay, symbol ROTARY-ENCODER-Ebay
- C1, C2, C3, C4, C7, C8: value 1u -> 47n
- D1, D2, D3, D4, D5, D6: footprint Diodes_SMD:D_MELF-RM10_Universal_Handsoldering -> Diodes_SMD:D_MiniMELF_Handsoldering
Connections:
- net GND: now also C11.2, ROT1.2 (C), ROT1.5 (SW1), ROT2.2 (C), ROT2.5 (SW1)
- net SCL: now also J2.1 (P1), Q2.2 (S), R15.2; no longer J3.4 (P4), Q2.3 (D), R16.2
- net SDA: now also J2.2 (P2), Q1.2 (S), R13.2; no longer J3.3 (P3), Q1.3 (D), R14.2
- net VCC: now also C11.1
- net VDD: now also J3.2 (P2)
- net enc1B: now also U1.4; no longer U1.6
- net enc1BTN: now also U1.6; no longer U1.4
- net enc2B: now also U1.10; no longer U1.12
- net enc2BTN: now also U1.12; no longer U1.10
- net at D4.2 (A), R8.2, R9.1: now also ROT2.3 (B)
- net at C3.2, D5.1 (K), R10.1: now also U1.13; no longer U1.11
- net at D6.2 (A), R11.2, R12.1: now also ROT2.1 (A)
- net at D5.2 (A), R10.2, R7.1: now also ROT2.4 (SW2)
- net at C4.2, D6.1 (K), R12.2: now also U1.11; no longer U1.13
- net at D1.2 (A), R2.2, R3.1: now also ROT1.3 (B)
- net at C1.2, D2.1 (K), R4.1: now also U1.5; no longer U1.3
- net at D3.2 (A), R5.2, R6.1: now also ROT1.1 (A)
- net at D2.2 (A), R1.1, R4.2: now also ROT1.4 (SW2)
- net at C2.2, D3.1 (K), R6.2: now also U1.3; no longer U1.5
- new net SCLlvl: J3.4 (P4), Q2.3 (D), R16.2
- new net SDAlvl: J3.3 (P3), Q1.3 (D), R14.2
Other:
- moved on the sheet: R1, U1B, U1C, U1E, U1F
